Commit message: lidar upgrade

File: description/aft_lidar.xacro (robot description, xacro)
@@ -1,10 +1,10 @@
 <?xml version="1.0"?>
-<robot xmlns:xacro="http://www.ros.org/wiki/xacro" >
-    <joint name="laser_joint" type="fixed">
+<robot xmlns:xacro="http://www.ros.org/wiki/xacro">
+    <joint name="aft_laser_joint" type="fixed">
         <parent link="chassis"/>
-        <child link="laser_frame"/>
-        <origin xyz="0.1 0 0.175" rpy="0 0 0"/>
+        <child link="aft_laser_frame"/>
+        <origin xyz="-1 0 0.175" rpy="0 0 0"/>
     </joint>
-    <link name="laser_frame">
+    <link name="aft_laser_frame">
         <visual>
             <geometry>
@@ -22,7 +22,7 @@
         </xacro:inertial_cylinder>
     </link>
-    <gazebo reference="laser_frame">
+    <gazebo reference="aft_laser_frame">
         <material>Gazebo/Red</material>
-        <sensor name="laser" type="ray">
+        <sensor name="aft_laser" type="ray">
             <pose> 0 0 0 0 0 0 </pose>
             <visualize>false</visualize>
@@ -41,10 +41,11 @@
                 </range>
             </ray>
-            <plugin name="laser_controller" filename="libgazebo_ros_ray_sensor.so">
+            <plugin name="aft_laser_controller" filename="libgazebo_ros_ray_sensor.so">
                 <ros>
-                    <argument>~/out:=scan</argument>
+                    <namespace>aft_laser</namespace>
+                    <remapping>~/out:=aft_scan</remapping>
                 </ros>
                 <output_type>sensor_msgs/LaserScan</output_type>
-                <frame_name>laser_frame</frame_name>
+                <frame_name>aft_laser_frame</frame_name>
             </plugin>
         </sensor>

File: description/robot.urdf.xacro (robot description, xacro)
@@ -3,5 +3,6 @@
     <xacro:include filename="robot_core.xacro" />
     <xacro:include filename="gazebo_control.xacro" />
-    <xacro:include filename="lidar.xacro" />
+    <xacro:include filename="front_lidar.xacro" />
+    <xacro:include filename="aft_lidar.xacro" />
     <xacro:include filename="camera.xacro" />
     <xacro:include filename="depth_camera.xacro" />
